File: arena_12_20_top/panels_ring_12_20_top.sch (KiCad schematic (older format))
At the start: 26 parts, among them P1 COLUMN_0, P10 COLUMN_9, P11 COLUMN_10, P12 COLUMN_11, P16 CONN_1, P17 CONN_1, P18 CONN_1, P19 CONN_1, P2 COLUMN_1, P20 CONN_1, P21 CONN_1, P22 CONN_1, P23 CONN_1, P24 CONN_1, P25 CONN_1, P26 CONN_1, P27 CONN_1, P28 CONN_1, P29 CONN_1, P3 COLUMN_2, P4 COLUMN_3, P5 COLUMN_4, P6 COLUMN_5, P7 COLUMN_6, P8 COLUMN_7, P9 COLUMN_8

Commit message: Finished Ver. 1 of panels_ring_12_20_top
Parts:
- removed P16, P17, P25: CONN_1, symbol CONN_1
- renumbered P26 to P25, P27 to P26, P28 to P27, P29 to P28
Connections:
- net GND: now reaches P7.8 (P8)
- net GND: now also P1.8 (P8), P10.8 (P8), P11.8 (P8), P12.8 (P8), P18.1, P19.1, P2.8 (P8), P20.1, P21.1, P22.1, P23.1, P24.1, P25.1, P26.1, P27.1, P28.1, P3.8 (P8), P4.8 (P8), P5.8 (P8), P6.8 (P8), P8.8 (P8), P9.8 (P8)
- no-connect marks 110 -> 84
Other:
- note removed: "1/4-20 mounting holes"
