File: arena_12_20_top/arena_12-20_top.sch (KiCad schematic (older format))
At the start: 25 parts, among them P1 COLUMN_0, P10 COLUMN_9, P11 COLUMN_10, P12 COLUMN_11, P16 CONN_1, P17 CONN_1, P18 CONN_1, P19 CONN_1, P2 COLUMN_1, P20 CONN_1, P21 CONN_1, P22 CONN_1, P23 CONN_1, P24 CONN_1, P25 CONN_1, P26 CONN_1, P27 CONN_1, P28 CONN_1, P3 COLUMN_2, P4 COLUMN_3, P5 COLUMN_4, P6 COLUMN_5, P7 COLUMN_6, P8 COLUMN_7, P9 COLUMN_8

Commit message: cleanup arena 12-20 top
Parts:
- removed P16, P17: CONN_1, symbol CONN_1
- P1, P10, P11, P12, P2, P3, P4, P5, P6, P7, P8, P9: symbol CONN_8 -> arena_12-20_top:CONN_8
- P18, P19, P20, P21, P22, P23, P24, P25, P26, P27, P28: symbol CONN_1 -> arena_12-20_top:CONN_1
Connections:
- net GND: no longer P28.1
Other:
- note removed: "1/4-20 mounting holes"
