File: arena_12_20/arena_12-20.sch (KiCad schematic (older format))
At the start: 32 parts, among them J1 DB9, P1 COLUMN_0, P10 COLUMN_9, P11 COLUMN_10, P12 COLUMN_11, P13 DIN_5, P14 CONN_5X2, P15 CONN_2, P16 CONN_1, P17 CONN_1, P18 CONN_1, P19 CONN_1, P2 COLUMN_1, P20 CONN_1, P21 CONN_1, P22 CONN_1, P23 CONN_1, P24 CONN_1, P25 CONN_1, P26 CONN_1, P27 CONN_1, P28 CONN_1, P3 COLUMN_2, P4 COLUMN_3, P5 COLUMN_4, P6 COLUMN_5, P7 COLUMN_6, P8 COLUMN_7, P9 COLUMN_8, SW1 SWITCH_INV

Commit message: start documentation of arena
Parts:
- C1, C2: symbol panels_ring_12_20:CAPAPOL -> arena_12-20:CAPAPOL
- J1: symbol panels_ring_12_20:DB9 -> arena_12-20:DB9
- P1, P10, P11, P12, P2, P3, P4, P5, P6, P7, P8, P9: symbol panels_ring_12_20:CONN_8 -> arena_12-20:CONN_8
- P13: symbol panels_ring_12_20:DIN_5 -> arena_12-20:DIN_5
- P14: symbol panels_ring_12_20:CONN_5X2 -> arena_12-20:CONN_5X2
- P15: symbol panels_ring_12_20:CONN_2 -> arena_12-20:CONN_2
- P16, P17, P18, P19, P20, P21, P22, P23, P24, P25, P26, P27, P28: symbol panels_ring_12_20:CONN_1 -> arena_12-20:CONN_1
- SW1: symbol panels_ring_12_20:SWITCH_INV -> arena_12-20:SWITCH_INV
Changed lines of the file:
@@
 	3900 3400 3700 3400
 $Comp
-L panels_ring_12_20:CONN_1 P28
+L arena_12-20:CONN_1 P28
 U 1 1 4D19112A
 P 4050 3400
@@
 $EndComp
 $Comp
-L panels_ring_12_20:CONN_1 P27
+L arena_12-20:CONN_1 P27
 U 1 1 4D191129
 P 4050 3200
@@
 $EndComp
 $Comp
-L panels_ring_12_20:CONN_1 P26
+L arena_12-20:CONN_1 P26
 U 1 1 4D191126
 P 4050 3000
@@
 $EndComp
 $Comp
-L panels_ring_12_20:CONN_1 P25
+L arena_12-20:CONN_1 P25
 U 1 1 4D191125
 P 4050 2800
@@
 $EndComp
 $Comp
-L panels_ring_12_20:CONN_1 P24
+L arena_12-20:CONN_1 P24
 U 1 1 4D19111C
 P 4050 2400
@@
 8-32 mounting holes
 $Comp
-L panels_ring_12_20:GND #PWR01
+L arena_12-20:GND #PWR01
 U 1 1 4D19062B
 P 2850 3700
@@
 $EndComp
 $Comp
-L panels_ring_12_20:CONN_1 P23
+L arena_12-20:CONN_1 P23
 U 1 1 4D1905C4
 P 3200 3400
@@
 $EndComp
 $Comp
-L panels_ring_12_20:CONN_1 P20
+L arena_12-20:CONN_1 P20
 U 1 1 4D1905C2
 P 3200 2800
@@
 $EndComp
 $Comp
-L panels_ring_12_20:CONN_1 P19
+L arena_12-20:CONN_1 P19
 U 1 1 4D1905C0
 P 3200 2600
@@
 $EndComp
 $Comp
-L panels_ring_12_20:CONN_1 P18
+L arena_12-20:CONN_1 P18
 U 1 1 4D1905BE
 P 3200 2400
@@
 $EndComp
 $Comp
-L panels_ring_12_20:CONN_1 P22
+L arena_12-20:CONN_1 P22
 U 1 1 4D1905BC
 P 3200 3200
@@
 $EndComp
 $Comp
-L panels_ring_12_20:CONN_1 P21
+L arena_12-20:CONN_1 P21
 U 1 1 4D1905B4
 P 3200 3000
@@
 NoConn ~ 2150 6150
 $Comp
-L panels_ring_12_20:SWITCH_INV SW1
+L arena_12-20:SWITCH_INV SW1
 U 1 1 4D13B1B5
 P 2650 6250
@@
 $EndComp
 $Comp
-L panels_ring_12_20:CONN_1 P17
+L arena_12-20:CONN_1 P17
 U 1 1 4D13AE2D
 P 3700 4200
@@
 $EndComp
 $Comp
-L panels_ring_12_20:CONN_1 P16
+L arena_12-20:CONN_1 P16
 U 1 1 4D13AE27
 P 3000 4200
@@
 $EndComp
 $Comp
-L panels_ring_12_20:GND #PWR04
+L arena_12-20:GND #PWR04
 U 1 1 4D12B446
 P 4150 7100
@@
 $EndComp
 $Comp
-L panels_ring_12_20:CONN_2 P15
+L arena_12-20:CONN_2 P15
 U 1 1 4D12B40B
 P 3650 6900
@@
 SCL_1
 $Comp
-L panels_ring_12_20:CONN_5X2 P14
+L arena_12-20:CONN_5X2 P14
 U 1 1 4D12B1EB
 P 3900 1300
@@
 $EndComp
 $Comp
-L panels_ring_12_20:GND #PWR06
+L arena_12-20:GND #PWR06
 U 1 1 4D12AF2A
 P 3550 4550
@@
 $EndComp
 $Comp
-L panels_ring_12_20:GND #PWR07
+L arena_12-20:GND #PWR07
 U 1 1 4D12AF26
 P 2850 4550
@@
 $EndComp
 $Comp
-L panels_ring_12_20:VCC #PWR08
+L arena_12-20:VCC #PWR08
 U 1 1 4D12AC6C
 P 9750 4350
@@
 $EndComp
 $Comp
-L panels_ring_12_20:VCC #PWR09
+L arena_12-20:VCC #PWR09
 U 1 1 4D12AC67
 P 8550 4350
@@
 $EndComp
 $Comp
-L panels_ring_12_20:VCC #PWR010
+L arena_12-20:VCC #PWR010
 U 1 1 4D12AC62
 P 7250 4350
@@
 $EndComp
 $Comp
-L panels_ring_12_20:VCC #PWR011
+L arena_12-20:VCC #PWR011
 U 1 1 4D12AC5C
 P 9750 3350
@@
 $EndComp
 $Comp
-L panels_ring_12_20:VCC #PWR012
+L arena_12-20:VCC #PWR012
 U 1 1 4D12AC58
 P 8550 3350
@@
 $EndComp
 $Comp
-L panels_ring_12_20:VCC #PWR013
+L arena_12-20:VCC #PWR013
 U 1 1 4D12AC53
 P 7250 3350
@@
 $EndComp
 $Comp
-L panels_ring_12_20:VCC #PWR014
+L arena_12-20:VCC #PWR014
 U 1 1 4D12AC4D
 P 9750 2400
@@
 $EndComp
 $Comp
-L panels_ring_12_20:VCC #PWR015
+L arena_12-20:VCC #PWR015
 U 1 1 4D12AC47
 P 8550 2400
@@
 $EndComp
 $Comp
-L panels_ring_12_20:VCC #PWR016
+L arena_12-20:VCC #PWR016
 U 1 1 4D12AC42
 P 7250 2400
@@
 $EndComp
 $Comp
-L panels_ring_12_20:VCC #PWR017
+L arena_12-20:VCC #PWR017
 U 1 1 4D12AC3D
 P 9750 1400
@@
 $EndComp
 $Comp
-L panels_ring_12_20:VCC #PWR018
+L arena_12-20:VCC #PWR018
 U 1 1 4D12AC37
 P 8550 1400
@@
 $EndComp
 $Comp
-L panels_ring_12_20:VCC #PWR019
+L arena_12-20:VCC #PWR019
 U 1 1 4D12AC18
 P 7250 1400
@@
 SCL_0
 $Comp
-L panels_ring_12_20:GND #PWR020
+L arena_12-20:GND #PWR020
 U 1 1 4D12A99C
 P 10150 5250
@@
 $EndComp
 $Comp
-L panels_ring_12_20:GND #PWR021
+L arena_12-20:GND #PWR021
 U 1 1 4D12A997
 P 8950 5250
@@
 $EndComp
 $Comp
-L panels_ring_12_20:GND #PWR022
+L arena_12-20:GND #PWR022
 U 1 1 4D12A993
 P 7650 5250
@@
 $EndComp
 $Comp
-L panels_ring_12_20:GND #PWR023
+L arena_12-20:GND #PWR023
 U 1 1 4D12A98C
 P 10150 4250
@@
 $EndComp
 $Comp
-L panels_ring_12_20:GND #PWR024
+L arena_12-20:GND #PWR024
 U 1 1 4D12A989
 P 8950 4250
@@
 $EndComp
 $Comp
-L panels_ring_12_20:GND #PWR025
+L arena_12-20:GND #PWR025
 U 1 1 4D12A983
 P 7650 4250
@@
 $EndComp
 $Comp
-L panels_ring_12_20:GND #PWR026
+L arena_12-20:GND #PWR026
 U 1 1 4D12A97B
 P 10150 3300
@@
 $EndComp
 $Comp
-L panels_ring_12_20:GND #PWR027
+L arena_12-20:GND #PWR027
 U 1 1 4D12A973
 P 8950 3300
@@
 $EndComp
 $Comp
-L panels_ring_12_20:GND #PWR028
+L arena_12-20:GND #PWR028
 U 1 1 4D12A96D
 P 7650 3300
@@
 $EndComp
 $Comp
-L panels_ring_12_20:GND #PWR029
+L arena_12-20:GND #PWR029
 U 1 1 4D12A95F
 P 10150 2300
@@
 $EndComp
 $Comp
-L panels_ring_12_20:GND #PWR030
+L arena_12-20:GND #PWR030
 U 1 1 4D12A950
 P 8950 2300
@@
 $EndComp
 $Comp
-L panels_ring_12_20:GND #PWR031
+L arena_12-20:GND #PWR031
 U 1 1 4D12A94E
 P 7650 2300
@@
 NoConn ~ 7750 1800
 $Comp
-L panels_ring_12_20:GND #PWR032
+L arena_12-20:GND #PWR032
 U 1 1 4D12A6CB
 P 6250 6600
@@
 $EndComp
 $Comp
-L panels_ring_12_20:GND #PWR033
+L arena_12-20:GND #PWR033
 U 1 1 4D12A6C8
 P 5300 6600
@@
 $EndComp
 $Comp
-L panels_ring_12_20:VCC #PWR034
+L arena_12-20:VCC #PWR034
 U 1 1 4D12A6C1
 P 6250 5900
@@
 $EndComp
 $Comp
-L panels_ring_12_20:VCC #PWR035
+L arena_12-20:VCC #PWR035
 U 1 1 4D12A6BC
 P 5300 5900
@@
 $EndComp
 $Comp
-L panels_ring_12_20:VCC #PWR036
+L arena_12-20:VCC #PWR036
 U 1 1 4D12A0AF
 P 3600 6100
@@
 $EndComp
 $Comp
-L panels_ring_12_20:GND #PWR037
+L arena_12-20:GND #PWR037
 U 1 1 4D12A09E
 P 1250 7100
@@
 SCL_1
 $Comp
-L panels_ring_12_20:CAPAPOL C2
+L arena_12-20:CAPAPOL C2
 U 1 1 4D129B77
 P 6250 6250
@@
 $EndComp
 $Comp
-L panels_ring_12_20:CAPAPOL C1
+L arena_12-20:CAPAPOL C1
 U 1 1 4D129B16
 P 5300 6250
@@
 $EndComp
 $Comp
-L panels_ring_12_20:DIN_5 P13
+L arena_12-20:DIN_5 P13
 U 1 1 4D129A69
 P 2000 6950
@@
 $EndComp
 $Comp
-L panels_ring_12_20:DB9 J1
+L arena_12-20:DB9 J1
 U 1 1 4D1299C1
 P 1500 1350
@@
 $EndComp
 $Comp
-L panels_ring_12_20:CONN_8 P3
+L arena_12-20:CONN_8 P3
 U 1 1 4D1299A0
 P 10600 1850
@@
 $EndComp
 $Comp
-L panels_ring_12_20:CONN_8 P6
+L arena_12-20:CONN_8 P6
 U 1 1 4D12999F
 P 10600 2850
@@
 $EndComp
 $Comp
-L panels_ring_12_20:CONN_8 P12
+L arena_12-20:CONN_8 P12
 U 1 1 4D12999E
 P 10600 4800
@@
 $EndComp
 $Comp
-L panels_ring_12_20:CONN_8 P9
+L arena_12-20:CONN_8 P9
 U 1 1 4D12999D
 P 10600 3800
@@
 $EndComp
 $Comp
-L panels_ring_12_20:CONN_8 P8
+L arena_12-20:CONN_8 P8
 U 1 1 4D129997
 P 9400 3800
@@
 $EndComp
 $Comp
-L panels_ring_12_20:CONN_8 P11
+L arena_12-20:CONN_8 P11
 U 1 1 4D129996
 P 9400 4800
@@
 $EndComp
 $Comp
-L panels_ring_12_20:CONN_8 P5
+L arena_12-20:CONN_8 P5
 U 1 1 4D129995
 P 9400 2850
@@
 $EndComp
 $Comp
-L panels_ring_12_20:CONN_8 P2
+L arena_12-20:CONN_8 P2
 U 1 1 4D129994
 P 9400 1850
@@
 $EndComp
 $Comp
-L panels_ring_12_20:CONN_8 P1
+L arena_12-20:CONN_8 P1
 U 1 1 4D12997C
 P 8100 1850
@@
 $EndComp
 $Comp
-L panels_ring_12_20:CONN_8 P4
+L arena_12-20:CONN_8 P4
 U 1 1 4D12997B
 P 8100 2850
@@
 $EndComp
 $Comp
-L panels_ring_12_20:CONN_8 P10
+L arena_12-20:CONN_8 P10
 U 1 1 4D12996A
 P 8100 4800
@@
 $EndComp
 $Comp
-L panels_ring_12_20:CONN_8 P7
+L arena_12-20:CONN_8 P7
 U 1 1 4D12995D
 P 8100 3800
