File: planar_arena_8x/arena_8-inf.sch (KiCad schematic (older format))
At the start: 22 parts, among them J1 DB9, P1 CONN_2, P10 CONN_8, P11 CONN_8, P12 CONN_8, P13 CONN_8, P14 CONN_8, P15 CONN_8, P16 CONN_8, P17 CONN_8, P2 CONN_4X2, P3 CONN_4X2, P4 CONN_4X2, P5 CONN_4X2, P6 CONN_4X2, P7 CONN_4X2, P8 CONN_4X2, P9 CONN_4X2, SW1 SWITCH_INV

Commit message: cleanup arena_8-inf
Parts:
- C1, C2, C3: symbol CP1 -> arena_8-inf:CP1
- J1: symbol DB9 -> arena_8-inf:DB9
- P1: symbol CONN_2 -> arena_8-inf:CONN_2
- P10, P11, P12, P13, P14, P15, P16, P17: symbol CONN_8 -> arena_8-inf:CONN_8
- P2, P3, P4, P5, P6, P7, P8, P9: symbol CONN_4X2 -> arena_8-inf:CONN_4X2
- SW1: symbol SWITCH_INV -> arena_8-inf:SWITCH_INV
